Commit message: leg config

File: description/urdf/awesome_leg_test_rig.urdf.xacro (robot description, xacro)
@@ -43,5 +43,5 @@
     </link>
     <xacro:if value="$(arg sliding_guide)">
-        <joint name="test_rig2base" type="prismatic">
+        <joint name="test_rig2base" type="fixed">
             <parent link="test_rig" />
             <child link="base_link" />

File: description/urdf/generated/awesome_leg.urdf (robot description, URDF)
Before this commit: robot awesome_leg, 6 links, 5 joints
Joints:
- joint test_rig2base: type prismatic -> fixed
